Commit message: tested with hw

File: musc_shoulder/model.urdf (robot description, URDF)
Before this commit: robot musc_shoulder, 4 links, 3 joints
Joints:
- joint axis1: limit lower=-1.57079632679 upper=1.57079632679 effort=0.0 velocity=0.0 -> lower=-0.4 upper=0.0 effort=0.0 velocity=0.0
- joint axis2: limit lower=-1.2217304764 upper=1.2217304764 effort=0.0 velocity=0.0 -> lower=-0.3 upper=0.0 effort=0.0 velocity=0.0

Commit message: correct joint limits & config

File: musc_shoulder/model.urdf (robot description, URDF)
Before this commit: robot musc_shoulder, 4 links, 3 joints
Joints:
- joint axis0: limit lower=0.0 upper=1.57079632679 effort=0.0 velocity=0.0 -> lower=0.0 upper=1.0 effort=0.0 velocity=0.0
- joint axis1: axis 1 0 0 -> -1 0 0; limit lower=-0.4 upper=0.0 effort=0.0 velocity=0.0 -> lower=0 upper=0.52 effort=0.0 velocity=0.0
- joint axis2: axis 0 0 1 -> 0 0 -1; limit lower=-0.3 upper=0.0 effort=0.0 velocity=0.0 -> lower=0 upper=0.26 effort=0.0 velocity=0.0

Commit message: adapted for bullet

File: musc_shoulder/model.urdf (robot description, URDF)
Before this commit: robot musc_shoulder, 4 links, 3 joints
Links:
- link arm: geometry collision mesh filename=meshes/CAD/arm.stl scale=0.001 0.001 0.001; visual mesh filename=meshes/CAD/arm.stl scale=0.001 0.001 0.001
- link base: geometry collision mesh filename=meshes/CAD/base.stl scale=0.001 0.001 0.001; visual mesh filename=meshes/CAD/base.stl scale=0.001 0.001 0.001
- link shoulder_link1: geometry collision mesh filename=meshes/CAD/shoulder_link1.stl scale=0.001 0.001 0.001; visual mesh filename=meshes/CAD/shoulder_link1.stl scale=0.001 0.001 0.001
- link shoulder_link2: geometry collision mesh filename=meshes/CAD/shoulder_link2.stl scale=0.001 0.001 0.001; visual mesh filename=meshes/CAD/shoulder_link2.stl scale=0.001 0.001 0.001
