Commit message: latest nano

File: upper_body/model.urdf (robot description, URDF)
Before this commit: robot upper_body, 14 links, 13 joints
Joints:
- joint elbow_left_axis0: limit lower=0.0 upper=0.9 effort=1.0 velocity=10.0 -> lower=0.0 upper=0.5 effort=1.0 velocity=10.0
- joint elbow_left_axis1: limit lower=0.0 upper=0.73 effort=1.0 velocity=10.0 -> lower=0.0 upper=0.5 effort=1.0 velocity=10.0
- joint elbow_right_axis0: limit lower=0.0 upper=0.9 effort=1.0 velocity=10.0 -> lower=0.0 upper=0.5 effort=1.0 velocity=10.0
- joint elbow_right_axis1: limit lower=0.0 upper=0.73 effort=1.0 velocity=10.0 -> lower=0.0 upper=0.5 effort=1.0 velocity=10.0

Commit message: fixed elbow joint limits

File: upper_body/model.urdf (robot description, URDF)
Before this commit: robot upper_body, 14 links, 13 joints
Joints:
- joint elbow_left_axis0: limit lower=0.0 upper=0.5 effort=1.0 velocity=10.0 -> lower=0.0 upper=0.9 effort=1.0 velocity=10.0
- joint elbow_left_axis1: limit lower=0.0 upper=0.5 effort=1.0 velocity=10.0 -> lower=0.0 upper=0.9 effort=1.0 velocity=10.0
- joint elbow_right_axis0: limit lower=0.0 upper=0.5 effort=1.0 velocity=10.0 -> lower=0.0 upper=0.9 effort=1.0 velocity=10.0
- joint elbow_right_axis1: limit lower=0.0 upper=0.5 effort=1.0 velocity=10.0 -> lower=0.0 upper=0.9 effort=1.0 velocity=10.0

Commit message: elbow limits corrected

File: upper_body/model.urdf (robot description, URDF)
Before this commit: robot upper_body, 14 links, 13 joints
Joints:
- joint elbow_left_axis0: limit lower=0.0 upper=0.9 effort=1.0 velocity=10.0 -> lower=0.0 upper=0.75 effort=1.0 velocity=10.0
- joint elbow_left_axis1: limit lower=0.0 upper=0.9 effort=1.0 velocity=10.0 -> lower=0.0 upper=0.75 effort=1.0 velocity=10.0
- joint elbow_right_axis0: limit lower=0.0 upper=0.9 effort=1.0 velocity=10.0 -> lower=0.0 upper=0.75 effort=1.0 velocity=10.0
- joint elbow_right_axis1: limit lower=0.0 upper=0.9 effort=1.0 velocity=10.0 -> lower=0.0 upper=0.75 effort=1.0 velocity=10.0

Commit message: took out shoulder axis2 rotation

File: upper_body/model.urdf (robot description, URDF)
Before this commit: robot upper_body, 14 links, 13 joints
Joints:
- joint shoulder_left_axis2: limit lower=-0.3 upper=0.3 effort=1.0 velocity=10.0 -> lower=0.0 upper=0.0 effort=1.0 velocity=10.0
- joint shoulder_right_axis2: limit lower=-0.3 upper=0.3 effort=0.0 velocity=0.0 -> lower=0.0 upper=0.0 effort=0.0 velocity=0.0
